File: hardware/HPM5E31.kicad_pcb (KiCad board)
At the start: 4 copper layers, 40 x 52 mm, 194 parts, among them J1 USB_C_Receptacle_USB2.0_16P, Q1 AGM60P100A, Q2 PMBT3904, Q3 PMBT3904, Q4 AO3404A, U10 TJA1042TK-3, U11 TJA1042TK-3, U12 TJA1042TK-3, U3 TJA1100HNZ, U4 RY3430, U5 LMR51450, U6 USBLC6-2SC6, U7 HPM5E3YIVK1, U8 ICM-42688P-HXY, U9 TJA1042TK-3, Y1 24M, Y3 25M

Commit message: Update HPM5E31 hardware design and manufacturing files
Parts:
- removed C10, C11, C8, C9: 10uF, Capacitor_SMD:C_0603_1608Metric
- removed C12: 4.7uF, Capacitor_SMD:C_0805_2012Metric
- removed C13, C14: 100nF, Capacitor_SMD:C_0603_1608Metric
- removed C15: 100nF, Capacitor_SMD:C_0805_2012Metric
- removed C16, C17: 22uF, Capacitor_SMD:C_0805_2012Metric
- removed C19: 10uF, Capacitor_SMD:C_0805_2012Metric
- removed C34, C57, C58, C59, C60, C61: 100nF, Capacitor_SMD:C_0402_1005Metric
- removed C55, C56: 12pF, Capacitor_SMD:C_0402_1005Metric
- removed C62, C63: 470nF, Capacitor_SMD:C_0402_1005Metric
- removed C77: 10nF, Capacitor_SMD:C_0402_1005Metric
- removed C86, C87: 10pF, Capacitor_SMD:C_0402_1005Metric
- removed D4: LED_E, LED_SMD:LED_0402_1005Metric
- removed D5: LED_G, LED_SMD:LED_0402_1005Metric
- removed KEY2: 笑脸开关3*5, Button_Switch_SMD:SW_Push_1P1T-MP_NO_Horizontal_Alps_SKRTLAE010
- removed L13: 3416自耦环, Inductor_SMD:L_CommonMode_Wurth_WE-CNSW-1206
- removed R11: 0R, Resistor_SMD:R_0603_1608Metric
- removed R27: 10K, Resistor_SMD:R_0402_1005Metric
- removed R35: 1K, Resistor_SMD:R_0402_1005Metric
- removed R4: 14.7K, Resistor_SMD:R_0402_1005Metric
- removed R5, R7: 100K, Resistor_SMD:R_0402_1005Metric
- removed R8: 19.1K, Resistor_SMD:R_0402_1005Metric
- removed Y3: 25M, Crystal:Crystal_SMD_2016-4Pin_2.0x1.6mm
- added C100: 100nF, Capacitor_SMD:C_0402_1005Metric, B.Cu at (71.4, 121.0)
- added C101: 100nF, Capacitor_SMD:C_0402_1005Metric, B.Cu at (74.7, 119.7)
- added C102: 100nF, Capacitor_SMD:C_0402_1005Metric, B.Cu at (72.9, 121.9)
- added C103: 100nF, Capacitor_SMD:C_0402_1005Metric, B.Cu at (71.4, 120.1)
- added C42: 10uF, Capacitor_SMD:C_0603_1608Metric, B.Cu at (75.5, 91.0)
- added C49: 100nF, Capacitor_SMD:C_0603_1608Metric, B.Cu at (70.5, 90.4)
- added C50: 22uF 10V, Capacitor_SMD:C_0805_2012Metric, B.Cu at (69.2, 85.5)
- added C51: 22uF 10V, Capacitor_SMD:C_0805_2012Metric, B.Cu at (66.3, 86.3)
- added C52: 22uF 10V, Capacitor_SMD:C_0805_2012Metric, B.Cu at (66.3, 101.7)
- added C53: 22uF 10V, Capacitor_SMD:C_0805_2012Metric, B.Cu at (64.3, 101.7)
- added C54: 100nF, Capacitor_SMD:C_0402_1005Metric, B.Cu at (75.2, 94.2)
- added C90: 100nF, Capacitor_SMD:C_0402_1005Metric, B.Cu at (88.3, 117.3)
- added C91: 100nF, Capacitor_SMD:C_0402_1005Metric, B.Cu at (87.0, 123.1)
- added C92: 100nF, Capacitor_SMD:C_0402_1005Metric, B.Cu at (85.6, 120.5)
- added C93: 100nF, Capacitor_SMD:C_0402_1005Metric, B.Cu at (82.9, 123.1)
- added C94: 100nF, Capacitor_SMD:C_0402_1005Metric, B.Cu at (84.9, 123.1)
- added C95: 100nF, Capacitor_SMD:C_0402_1005Metric, B.Cu at (86.0, 123.1)
- added C96: 100nF, Capacitor_SMD:C_0402_1005Metric, B.Cu at (85.6, 121.5)
- added C97: 100nF, Capacitor_SMD:C_0402_1005Metric, B.Cu at (83.9, 123.1)
- added C98: 470nF, Capacitor_SMD:C_0402_1005Metric, F.Cu at (86.5, 124.5)
- added C99: 100nF, Capacitor_SMD:C_0402_1005Metric, B.Cu at (73.9, 121.8)
- added D13: ESD9B5.0ST5G, Diode_SMD:D_SOD-923, F.Cu at (77.5, 101.4)
- added D17: ESD9B5.0ST5G, Diode_SMD:D_SOD-923, F.Cu at (74.6, 101.5)
- added D18: ESD9B5.0ST5G, Diode_SMD:D_SOD-923, B.Cu at (61.9, 123.3)
- added D19: ESD9B5.0ST5G, Diode_SMD:D_SOD-923, B.Cu at (61.8, 126.2)
- added D6: LED_G, LED_SMD:LED_0402_1005Metric, F.Cu at (68.1, 128.1)
- added D7: LED_E, LED_SMD:LED_0402_1005Metric, F.Cu at (66.1, 126.1)
- added D8: LED_G, LED_SMD:LED_0402_1005Metric, F.Cu at (65.1, 126.2)
- added F17: SMD0402, Fuse:Fuse_0402_1005Metric, F.Cu at (76.6, 101.4)
- added F18: SMD0402, Fuse:Fuse_0402_1005Metric, F.Cu at (75.5, 101.4)
- added F19: SMD0402, Fuse:Fuse_0402_1005Metric, B.Cu at (61.8, 124.2)
- added F22: SMD0402, Fuse:Fuse_0402_1005Metric, B.Cu at (61.8, 125.2)
- added G***: LOGO, LOGO, F.Cu at (79.1, 125.4)
- added G***: LOGO, LOGO, F.Cu at (92.8, 106.4)
- added H10: ~, Connector_JST:JST_GH_BM04B-GHS-TBT_1x04-1MP_P1.25mm_Vertical, F.Cu at (61.1, 106.9)
- added H11: ~, Connector_JST:JST_GH_BM04B-GHS-TBT_1x04-1MP_P1.25mm_Vertical, F.Cu at (79.4, 96.9)
- added H12: ~, Connector_JST:JST_GH_BM04B-GHS-TBT_1x04-1MP_P1.25mm_Vertical, F.Cu at (61.1, 125.8)
- added H13: MountingHole_Pad_MP, MountingHole:MountingHole_2.2mm_M2_DIN965_Pad, F.Cu at (66.6, 132.7)
- added H14: MountingHole_Pad_MP, MountingHole:MountingHole_2.2mm_M2_DIN965_Pad, F.Cu at (92.2, 132.7)
- added H15: MountingHole_Pad_MP, MountingHole:MountingHole_2.2mm_M2_DIN965_Pad, F.Cu at (60.3, 99.5)
- added H16: MountingHole_Pad_MP, MountingHole:MountingHole_2.2mm_M2_DIN965_Pad, F.Cu at (98.5, 99.5)
- added R14: 270K, Resistor_SMD:R_0603_1608Metric, B.Cu at (71.1, 86.9)
- added R17: 51K, Resistor_SMD:R_0603_1608Metric, B.Cu at (72.6, 86.9)
- added R18: 10R, Resistor_SMD:R_0402_1005Metric, F.Cu at (89.5, 109.1)
- added R36: 4.7K, Resistor_SMD:R_0402_1005Metric, F.Cu at (68.1, 126.2)
- added R37: 330R, Resistor_SMD:R_0402_1005Metric, F.Cu at (67.1, 128.0)
- added R41: 4.7K, Resistor_SMD:R_0402_1005Metric, F.Cu at (66.6, 124.7)
- added R42: 330R, Resistor_SMD:R_0402_1005Metric, F.Cu at (67.0, 126.1)
- added R43: 10K, Resistor_SMD:R_0402_1005Metric, B.Cu at (91.4, 121.4)
- added R44: 10K, Resistor_SMD:R_0402_1005Metric, B.Cu at (90.4, 121.4)
- added R45: 10K, Resistor_SMD:R_0402_1005Metric, B.Cu at (87.9, 119.1)
- added R46: 10K, Resistor_SMD:R_0402_1005Metric, B.Cu at (88.9, 119.1)
- added R47: 10K, Resistor_SMD:R_0402_1005Metric, B.Cu at (87.9, 121.1)
- added R52: 10K, Resistor_SMD:R_0402_1005Metric, B.Cu at (88.9, 121.1)
- added R53: 10K, Resistor_SMD:R_0402_1005Metric, F.Cu at (81.2, 120.7)
- added R54: 10K, Resistor_SMD:R_0402_1005Metric, F.Cu at (81.2, 122.0)
- added R55: 10K, Resistor_SMD:R_0402_1005Metric, B.Cu at (83.2, 115.9)
- added R56: 10K, Resistor_SMD:R_0402_1005Metric, B.Cu at (83.9, 115.2)
- added R57: 2.49K, Resistor_SMD:R_0402_1005Metric, F.Cu at (68.4, 123.0)
- added R58: 10K, Resistor_SMD:R_0402_1005Metric, F.Cu at (90.3, 123.2)
- added R59: 10K, Resistor_SMD:R_0402_1005Metric, F.Cu at (89.4, 124.4)
- added R60: 10K, Resistor_SMD:R_0402_1005Metric, F.Cu at (76.3, 123.2)
- added R61: 4.7K, Resistor_SMD:R_0402_1005Metric, F.Cu at (66.0, 128.1)
- added R62: 330R, Resistor_SMD:R_0402_1005Metric, F.Cu at (65.1, 128.1)
- added R63: 10K, Resistor_SMD:R_0402_1005Metric, B.Cu at (73.0, 115.0)
- added U14: HPM5E31IGN1, Library:BGA-196_14x14_12.0x12.0mm_P0.8mm, F.Cu at (79.4, 110.6)
- added U2: TJA1101B, Package_DFN_QFN:QFN-36-1EP_6x6mm_P0.5mm_EP4.1x4.1mm, F.Cu at (86.1, 120.3)
- C18, C20: footprint Capacitor_SMD:C_0805_2012Metric -> Capacitor_SMD:C_0603_1608Metric; moved to B.Cu
- C29, C64, C68, C69, C78, C79, C82, C83, L4, L5, L6, R48, U9: moved to F.Cu
- C36, C4, C43, C44, C6, C67, C7, C71, C72, C73, C75, C76, D11, D12, D14, D16, D25, D9, F13, F14, F15, F16, F3, F4, L1, L10, L11, L8, L9, Q4, R13, R15, R16, R2, R20, R22, R26, R3, R31, R32, R33, R34, R38, R39, R40, RR1, U4: moved to B.Cu
- C37: value 4.7uF -> 10uF; moved to B.Cu
- C39: value 4.7uF -> 10uF
- D1: footprint Diode_SMD:D_SMB -> Diode_SMD:D_SMA
- H3: footprint Connector_JST:JST_PH_B4B-PH-K_1x04_P2.00mm_Vertical -> Connector_JST:JST_GH_BM04B-GHS-TBT_1x04-1MP_P1.25mm_Vertical
- H4: footprint Connector_JST:JST_PH_B2B-PH-K_1x02_P2.00mm_Vertical -> Connector_JST:JST_GH_BM02B-GHS-TBT_1x02-1MP_P1.25mm_Vertical
- L12: footprint Inductor_SMD:L_CommonModeChoke_Coilcraft_0805USB -> Inductor_SMD:L_CommonModeChoke_Coilcraft_1812CAN
- L2: value 5.6uH -> 4.7uH; footprint Inductor_SMD:L_APV_APH0630 -> Inductor_SMD:L_APV_APH0420; moved to B.Cu
- Q2: footprint Package_TO_SOT_SMD:SOT-23 -> Package_TO_SOT_SMD:SOT-23-3
- U3: value TJA1100HNZ -> RTL8201F-VB-CG; footprint kicad_api_lib:TJA1100HNZ -> kicad_api_lib:RTL8201F-VB-CG; moved to F.Cu
- U5: value LMR51450 -> RY8411; footprint Package_SON:WSON-12-1EP_3x3mm_P0.5mm_EP1.5x2.5mm -> Package_TO_SOT_SMD:SOT-23-6; moved to B.Cu
- U7: value HPM5E3YIVK1 -> W25Q128JVS; footprint Library:BGA-121_11x11_9.0x9.0mm_P0.8mm -> Package_SO:SOIC-8_5.3x5.3mm_P1.27mm; moved to B.Cu
- moved L2 136.0 mm to (67.4, 90.3), turned to 90 degrees
- moved C20 123.9 mm to (77.0, 91.0), turned to 90 degrees
- moved C18 118.6 mm to (78.4, 91.0), turned to 90 degrees
- moved U5 113.6 mm to (72.9, 90.6), turned to -90 degrees
- moved C43 90.6 mm to (81.9, 116.5), turned to -135 degrees
- moved C44 89.3 mm to (82.5, 117.2), turned to -135 degrees
- moved C4 84.4 mm to (80.0, 115.1), turned to -45 degrees
- moved C72 82.2 mm to (94.2, 109.2), turned to -90 degrees
- moved C73 81.1 mm to (93.2, 109.2), turned to -90 degrees
- moved D15 81.1 mm to (60.5, 132.6), turned to 0 degrees
- moved C36 79.1 mm to (73.7, 111.2), turned to -45 degrees
- moved C76 77.4 mm to (60.5, 131.8)
- moved R40 77.0 mm to (98.5, 105.7), turned to 90 degrees
- moved C37 76.5 mm to (74.4, 110.6), turned to -45 degrees
- moved R15 74.4 mm to (78.0, 123.7), turned to -90 degrees
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Connections:
- C18 pad 1: +5V -> VIN
- C20 pad 1: +5V -> VIN
- C21 pad 1: +3.3V -> 3.3V
- C22 pad 1: +3.3V -> 3.3V
- C23 pad 1: +3.3V -> 3.3V
- C26 pad 1: Net-(C26-Pad1) -> +1V2
- C28 pad 1: Net-(C26-Pad1) -> +1V2
- C29 pad 1: Net-(C26-Pad1) -> +1V2
- C32 pad 2: Net-(U7C-VDD_OTPCAP) -> Net-(U14J-VDD_PMCCAP)
- C33 pad 2: Net-(U7C-VDD_OTPCAP) -> Net-(U14J-VDD_PMCCAP)
- C35 pad 2: Net-(U7C-VDD_PMCCAP) -> Net-(U14J-VDD_OTPCAP)
- C36 pad 2: Net-(U7C-VDD_PHY0CAP) -> Net-(U14J-VDD_PHY0CAP)
- C37 pad 2: Net-(U7C-VDD_PHY0CAP) -> Net-(U14J-VDD_PHY0CAP)
- C38 pad 2: Net-(U7C-VDD_PHY1CAP) -> Net-(U14J-VDD_PHY1CAP)
- C39 pad 2: Net-(U7C-VDD_PHY1CAP) -> Net-(U14J-VDD_PHY1CAP)
- C40 pad 1: Net-(U7C-XTALO) -> Net-(U14C-XTALO)
- C41 pad 2: Net-(U7C-XTALI) -> Net-(U14C-XTALI)
- C43 pad 2: +3.3V -> 3.3V
- C44 pad 2: +3.3V -> 3.3V
- C45 pad 2: +3.3V -> 3.3V
- C46 pad 2: +3.3V -> 3.3V
- C47 pad 2: +3.3V -> 3.3V
- C48 pad 2: +3.3V -> 3.3V
- C74 pad 1: 3.3V -> +5V
- C76 pad 1: User_Key -> +5V
- C78 pad 1: RD_P -> MDI+1
- C79 pad 1: RD_N -> MDI-1
- C80 pad 1: RD_P -> MDI-1
- C81 pad 1: RD_N -> MDI+1
- C82 pad 1: TD_N -> MDI-0
- C83 pad 1: TD_P -> MDI+0
- C84 pad 1: TD_P -> MDI-0
- C85 pad 1: TD_N -> MDI+0
- C88 pad 1: TRX_M -> Net-(C88-Pad1)
- C88 pad 2: Net-(C88-Pad2) -> TX_P
- C89 pad 1: TRX_P -> Net-(C89-Pad1)
- C89 pad 2: Net-(C89-Pad2) -> RX_N
- D10 pad 1: 3.3V -> +5V
- D11 pad 2: UART4_RX -> UART6_TX
- D12 pad 2: UART4_TX -> UART6_RX
- D14 pad 2: UART6_RX -> UART4_RX
- D15 pad 4: PWM0_P6 -> PWM0_P2
- D16 pad 2: UART6_TX -> UART4_TX
- D29 pad 2: UART0_TX -> UART0_RX
- D30 pad 2: UART0_RX -> UART0_TX
- F13 pad 1: UART6_TX -> UART4_TX
- F14 pad 1: UART6_RX -> UART4_RX
- F15 pad 1: UART4_RX -> UART6_TX
- F16 pad 1: UART4_TX -> UART6_RX
- F20 pad 2: UART0_RX -> UART0_TX
- F21 pad 2: UART0_TX -> UART0_RX
- F3 pad 1: Net-(D25-K-Pad2) -> Net-(D25-K-Pad1)
- F4 pad 1: Net-(D25-K-Pad1) -> Net-(D25-K-Pad2)
- H1 pad 2: Net-(F15-Pad2) -> +5V
- H1 pad 3: Net-(F16-Pad2) -> DBUS
- H2 pad 2: +5V -> UART1_TX
- H2 pad 3: DBUS -> UART1_RX
- H4 pad 1: Net-(H4-Pad1) -> RX_N
- H4 pad 2: Net-(H4-Pad2) -> TX_P
- J1 pad SH: (no net) -> GND
- L1 pad 2: +3.3V -> 3.3V
- L12 pad 1: Net-(C89-Pad2) -> TRX_P
- L12 pad 2: Net-(H4-Pad1) -> TRX_N
- L12 pad 3: Net-(H4-Pad2) -> Net-(C89-Pad1)
- L12 pad 4: Net-(C88-Pad2) -> Net-(C88-Pad1)
- L2 pad 1: Net-(C14-Pad2) -> Net-(U5-LX)
- L3 pad 1: Net-(C26-Pad1) -> +1V2
- L5 pad 1: Net-(U10-CANH) -> Net-(U10-CANL)
- L5 pad 2: Net-(U10-CANL) -> Net-(U10-CANH)
- L5 pad 3: Net-(D23-K-Pad2) -> Net-(D23-K-Pad1)
- L5 pad 4: Net-(D23-K-Pad1) -> Net-(D23-K-Pad2)
- L6 pad 1: Net-(U11-CANH) -> Net-(U11-CANL)
- L6 pad 2: Net-(U11-CANL) -> Net-(U11-CANH)
- L6 pad 3: Net-(D24-K-Pad2) -> Net-(D24-K-Pad1)
- L6 pad 4: Net-(D24-K-Pad1) -> Net-(D24-K-Pad2)
- L7 pad 3: Net-(D25-K-Pad1) -> Net-(D25-K-Pad2)
- L7 pad 4: Net-(D25-K-Pad2) -> Net-(D25-K-Pad1)
- L9 pad 1: Net-(C80-Pad2) -> Net-(C81-Pad2)
- L9 pad 4: Net-(C81-Pad2) -> Net-(C80-Pad2)
- MLT-1 pad 1: 3.3V -> +5V
- Q2 pad 3: UART2_RX -> UART5_RX
- Q3 pad 1: Net-(Q3-B) -> unconnected-(Q3-B-Pad1)
- R12 pad 1: Net-(U7C-XTALI) -> Net-(U14C-XTALI)
- R12 pad 2: Net-(U7C-XTALO) -> Net-(U14C-XTALO)
- R13 pad 1: Net-(U7C-WKUP) -> Net-(U14C-WKUP)
- R15 pad 1: ETH0_MDIO -> ESC0_MDIO
- R16 pad 1: ETH0_MDC -> ESC0_MDC
- R24 pad 1: UART2_RX -> UART5_RX
- R24 pad 2: +3.3V -> 3.3V
- R25 pad 1: 3.3V -> GND
- R25 pad 2: Net-(U3-EN/TXCLK) -> BOOT0
- R26 pad 1: 3.3V -> GND
- R26 pad 2: Net-(U3-TXER) -> BOOT1
- R28 pad 1: 3.3V -> ESC0_P1_RXD3
- R28 pad 2: INT_N -> GND
- R29 pad 1: Net-(Q3-B) -> Net-(R29-Pad1)
- R29 pad 2: PWM0_P2 -> PWM0_P1
- R3 pad 1: +3.3V -> 3.3V
- R30 pad 1: Net-(Q3-B) -> Net-(R29-Pad1)
- R31 pad 1: JTAG_TDI -> JTAG_TMS
- R31 pad 2: +3.3V -> 3.3V
- R32 pad 1: JTAG_TMS -> JTAG_TDI
- R32 pad 2: +3.3V -> 3.3V
- R34 pad 1: User_Key -> SPI2_CS
- R38 pad 2: PWM0_P3 -> PWM0_P4
- R39 pad 2: PWM0_P3 -> PWM0_P4
- U1 pad 1: JTAG_TDI -> Net-(F21-Pad1)
- U1 pad 2: JTAG_TMS -> Net-(F20-Pad1)
- U1 pad 3: JTAG_TCK -> JTAG_TDI
- U1 pad 4: JTAG_TRST -> JTAG_TDO
- U1 pad 5: JTAG_TDO -> JTAG_TRST
- U1 pad 6: Net-(F20-Pad1) -> JTAG_TMS
- U1 pad 7: Net-(F21-Pad1) -> JTAG_TCK
- U1 pad 9: +3.3V -> 3.3V
- U3 pad 1: ESC0_MDC -> Net-(U3-RSET)
- U3 pad 10: unconnected-(U3-INH-Pad10) -> ESC0_P0_RXD1
- U3 pad 11: 3.3V -> ESC0_P0_RXD2
- U3 pad 12: TRX_P -> ESC0_P0_RXD3
- U3 pad 13: TRX_M -> ESC0_P0_RXCK
- U3 pad 15: GND -> ESC0_P0_TXCK
- U3 pad 16: Net-(U3-VDDD(1V8)) -> ESC0_P0_TXD0
- U3 pad 17: ESC0_P1_RXER -> ESC0_P0_TXD1
- U3 pad 18: ESC0_P1_RXDV -> ESC0_P0_TXD2
- U3 pad 19: 3.3V -> ESC0_P0_TXD3
- U3 pad 2: INT_N -> Net-(U3-AVDD10OUT)
- U3 pad 20: GND -> ESC0_P0_TXEN
- U3 pad 21: ESC0_P1_RXD3 -> PHYRSTB
- U3 pad 22: ESC0_P1_RXD2 -> ESC0_MDC
- U3 pad 23: ESC0_P1_RXD1 -> ESC0_MDIO
- U3 pad 24: ESC0_P1_RXD0 -> ENET_PHY_LED0
- U3 pad 25: ESC0_P1_RXCK -> ENET_PHY_LED1
- U3 pad 26: GND -> CRS
- U3 pad 27: 3.3V -> COL
- U3 pad 28: ESC0_P1_TXCK -> ESC0_P0_RXER
- U3 pad 29: ESC0_P1_TXEN -> Net-(U3-DVDD10OUT)
- U3 pad 3: RST_N -> MDI+0
- U3 pad 30: ESC0_P1_TXD3 -> 3.3V
- U3 pad 31: ESC0_P1_TXD2 -> GND
- U3 pad 32: ESC0_P1_TXD1 -> ESC0_REFCK
- U3 pad 33: ESC0_P1_TXD0 -> GND
- U3 pad 4: Net-(U3-VDDA(1V8)) -> MDI-0
- U3 pad 5: Net-(U3-XO) -> MDI+1
- U3 pad 6: Net-(U3-XI) -> MDI-1
- U3 pad 8: Net-(D4-A) -> ESC0_P0_RXDV
- U3 pad 9: 3.3V -> ESC0_P0_RXD0
- U5 pad 1: Net-(C14-Pad2) -> Net-(U5-BS)
- U5 pad 2: Net-(C14-Pad2) -> GND
- U5 pad 3: Net-(C14-Pad2) -> Net-(U5-FB)
- U5 pad 4: Net-(U5-BOOT) -> VIN
- U5 pad 5: Net-(U5-PG) -> VIN
- U5 pad 6: Net-(U5-RT) -> Net-(U5-LX)
- U8 pad 1: SPI1_MISO -> SPI3_MISO
- U8 pad 12: SPI1_CS -> SPI3_CS
- U8 pad 13: SPI1_SCLK -> SPI3_SCLK
- U8 pad 14: SPI1_MOSI -> SPI3_MOSI
- Y1 pad 1: Net-(U7C-XTALO) -> Net-(U14C-XTALO)
- Y1 pad 3: Net-(U7C-XTALI) -> Net-(U14C-XTALI)
Routing:
- net 3.3V: track 0.00 -> 155.2 mm, vias 0 -> 34
- net GND: track 0.75 -> 110.5 mm, vias 2 -> 137
- net +5V: track 0.00 -> 70.2 mm, vias 0 -> 18
- net ESC0_REFCK: track 0.00 -> 34.1 mm, vias 0 -> 3
- net ESC0_MDIO: track 0.78 -> 34.6 mm, vias 1 -> 4
- net UART3_TX: track 0.00 -> 33.5 mm, vias 0 -> 1
- net ESC0_MDC: track 0.56 -> 33.4 mm, vias 1 -> 4
- net UART3_RX: track 0.00 -> 32.8 mm, vias 0 -> 1
- net PWM0_P1: track 0.00 -> 32.2 mm, vias 0 -> 3
- net RESET: track 0.46 -> 30.3 mm, vias 1 -> 2
- net UART5_RX: track 0.00 -> 27.7 mm, vias 0 -> 2
- net +1V2: track 0.00 -> 27.3 mm, vias 0 -> 5
- net COL: track 0.00 -> 26.4 mm, vias 0 -> 2
- net VBUS: track 0.00 -> 25.7 mm, vias 0 -> 1
- net CAN1_RXD: track 0.60 -> 25.7 mm, vias 1 -> 2
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- added copper zone on B.Cu, net +5V
- added copper zone on In2.Cu, net +5V
- added copper zone on B.Cu, net 3.3V
- added copper zone on In2.Cu, net 3.3V
- added copper zone on B.Cu, net GND
- added copper zone on F.Cu, net GND
- added copper zone on In1.Cu, net GND
- added copper zone on F.Cu, net VIN
- added copper zone on F.Cu, net VIN1
- removed copper zone on B.Cu, net Net-(L3-Pad2)
Other:
- board size 40 x 52 mm -> 42.7 x 52 mm
- board text added: "0"
- board text added: "1"
- board text added: "2"
- board text added: "3"
- board text added: "5 3 G TCK TMS RST TOD TDI TX RX"
- board text added: "5 G T R"
- board text added: "D 5 G"
- board text added: "DUST"
- board text added: "H L"
- board text added: "R T G"
- board text added: "R T G 5"
- board text added: "RESET"
- board text added: "TXD TXP RXD RXP"
- board text added: "TXP RXN"
