File: hardware/HPM5E31.kicad_sch (KiCad schematic)
At the start: 51 parts, among them Q1 AGM60P100A, U4 RY3430, U5 LMR51450, U7 HPM5E3YIVK1

Commit message: Update HPM5E31 hardware design and manufacturing files
Parts:
- removed C10, C11, C8, C9: 10uF, Capacitor_SMD:C_0603_1608Metric, symbol SparkFun-Capacitor:C_Small
- removed C12: 4.7uF, Capacitor_SMD:C_0805_2012Metric, symbol SparkFun-Capacitor:C
- removed C13, C14: 100nF, Capacitor_SMD:C_0603_1608Metric, symbol SparkFun-Capacitor:C
- removed C15: 100nF, Capacitor_SMD:C_0805_2012Metric, symbol SparkFun-Capacitor:C
- removed C16, C17: 22uF, Capacitor_SMD:C_0805_2012Metric, symbol SparkFun-Capacitor:C_Small
- removed C18, C19, C20: 10uF, Capacitor_SMD:C_0805_2012Metric, symbol SparkFun-Capacitor:C_Small
- removed L2: 5.6uH, Inductor_SMD:L_APV_APH0630, symbol SparkFun-Coil:L
- removed R11: 0R, Resistor_SMD:R_0603_1608Metric, symbol Device:R_Small
- removed R4: 14.7K, Resistor_SMD:R_0402_1005Metric, symbol Device:R_Small
- removed R5, R7: 100K, Resistor_SMD:R_0402_1005Metric, symbol Device:R_Small
- removed R8: 19.1K, Resistor_SMD:R_0402_1005Metric, symbol Device:R_Small
- removed U5: LMR51450, Package_SON:WSON-12-1EP_3x3mm_P0.5mm_EP1.5x2.5mm, symbol New_Library_0:TPS56637
- removed U7: HPM5E3YIVK1, Library:BGA-121_11x11_9.0x9.0mm_P0.8mm, symbol HPM5E00_Library:HPM5E3YIVK1
- added C18, C20, C42: 10uF, Capacitor_SMD:C_0603_1608Metric, symbol Device:C_Small
- added C49: 100nF, Capacitor_SMD:C_0603_1608Metric, symbol Device:C_Small
- added C50, C51, C52, C53: 22uF 10V, Capacitor_SMD:C_0805_2012Metric, symbol Device:C_Small
- added L2: 4.7uH, Inductor_SMD:L_APV_APH0420, symbol Device:L
- added R14: 270K, Resistor_SMD:R_0603_1608Metric, symbol Device:R
- added R17: 51K, Resistor_SMD:R_0603_1608Metric, symbol Device:R
- added U14: HPM5E31IGN1, HPM_footprints:BGA-196_14x14_12.0x12.0mm_P0.8mm, symbol HPM5E00_Library:HPM5E31IGN1
- added U5: RY8411, Package_TO_SOT_SMD:SOT-23-6, symbol 0_RM2023:SY8301
- C21, C22, C29, C45, C46, C47, C48: footprint Capacitor_SMD:C_0402_1005Metric -> SparkFun-Capacitor:C_0603_1608Metric
- C23: footprint Capacitor_SMD:C_0402_1005Metric -> SparkFun-Capacitor:C_0603_1608Metric; Voltage (none) -> 1kV
- C24, C25, C27, C30, C31: footprint Capacitor_SMD:C_0402_1005Metric -> SparkFun-Capacitor:C_0603_1608Metric; PROD_ID (none) -> CAP-00000; Tolerance (none) -> 100%; Voltage (none) -> 1kV
- C26, C28, C6, C7: footprint Capacitor_SMD:C_0603_1608Metric -> SparkFun-Capacitor:C_0603_1608Metric
- D1: footprint Diode_SMD:D_SMB -> Diode_SMD:D_SMA
- D3: footprint LED_SMD:LED_0603_1608Metric -> SparkFun-LED:LED_0603_1608Metric_Blue
Connections:
- net +1V2: now also C26.1, C28.1, C29.1, L3.1, U14.F6 (VDD_SOC), U14.F9 (VDD_SOC), U14.G6 (VDD_SOC), U14.G9 (VDD_SOC), U14.H9 (VDD_SOC)
- net +5V: now also C50.1, C51.1, L2.2, R14.2
- net GND: now also C18.2, C20.2, C42.2, C50.2, C51.2, C52.2, C53.2, R17.1, U14.A1 (VSS), U14.A14 (VSS), U14.E10 (VSS), U14.E5 (VSS), U14.F7 (VSS), U14.F8 (VSS), U14.G7 (VSS), U14.G8 (VSS), U14.H7 (VSS), U14.H8 (VSSA), U14.J7 (VSS), U14.J8 (VREFL), U14.K10 (VSS), U14.K5 (VSS), U14.N1 (DCDC_GND), U14.N3 (VSS), U14.P1 (VSS), U14.P14 (VSS), U14.P2 (DCDC_GND), U5.2 (GND)
- net VIN: now also C18.1, C20.1, C42.1, U5.4 (EN), U5.5 (IN)
- net at L3.2: now also U14.N2 (DCDC_LP), U14.P3 (DCDC_LP)
- net +3.3V renamed 3.3V
- net 3.3V: now also C52.1, C53.1, U14.J9 (VANA), U14.K9 (VREFH), U14.M1 (DCDC_IN), U14.M2 (DCDC_IN)
- new net: C49.1, L2.1, U5.6 (LX)
- new net: C49.2, U5.1 (BS)
- new net: R14.1, R17.2, U5.3 (FB)
