File: hardware/other.kicad_sch (KiCad schematic)
At the start: 77 parts, among them Q2 PMBT3904, Q3 PMBT3904, Q4 AO3404A, U10 TJA1042TK-3, U11 TJA1042TK-3, U12 TJA1042TK-3, U8 ICM-42688P-HXY, U9 TJA1042TK-3

Commit message: Update HPM5E31 hardware design and manufacturing files
Parts:
- removed C76: 100nF, Capacitor_SMD:C_0402_1005Metric, symbol SparkFun-Capacitor:C_Small
- removed KEY2: 笑脸开关3*5, Button_Switch_SMD:SW_Push_1P1T-MP_NO_Horizontal_Alps_SKRTLAE010, symbol New_Library_0:笑脸开关3*5
- added C54: 100nF, SparkFun-Capacitor:C_0603_1608Metric, symbol SparkFun-Capacitor:C_Small
- added D13, D17, D18, D19: ESD9B5.0ST5G, Diode_SMD:D_SOD-923, symbol Diode:ESD9B5.0ST5G
- added F17, F18, F19, F22: SMD0402, SparkFun-Fuse:Fuseholder_Automotive, symbol SparkFun-Fuse:Fuse_Holder-Blade
- added H10, H11, H12: (no value), Connector_JST:JST_GH_BM04B-GHS-TBT_1x04-1MP_P1.25mm_Vertical, symbol GH1.25:GH1.25_4P
- added H13, H14, H15, H16: MountingHole_Pad_MP, MountingHole:MountingHole_2.2mm_M2_DIN965_Pad, symbol Mechanical:MountingHole_Pad_MP
- added R25, R26: 10K, Resistor_SMD:R_0402_1005Metric, symbol Device:R_Small
- added U7: W25Q128JVS, Package_SO:SOIC-8_5.3x5.3mm_P1.27mm, symbol Memory_Flash:W25Q128JVS
- C64, C65, C66, C67, C68, C69, C70, C71, C72, C73, C74, C75: footprint Capacitor_SMD:C_0402_1005Metric -> SparkFun-Capacitor:C_0603_1608Metric
- D15: footprint LED_SMD:LED_WS2812B-Mini_PLCC4_3.5x3.5mm -> SparkFun-LED:WS2812_2020
- F10, F3, F4, F5, F6, F7, F8, F9: footprint Fuse:Fuse_0603_1608Metric -> SparkFun-Fuse:Fuseholder_Automotive
- F13, F14, F15, F16, F20, F21: footprint Fuse:Fuse_0402_1005Metric -> SparkFun-Fuse:Fuseholder_Automotive
- MLT-1: footprint Library:BUZ-SMD_L5.0-W5.5-P4.60 -> 蜂鸣器:
- Q2, Q3: footprint Package_TO_SOT_SMD:SOT-23 -> SparkFun-Semiconductor-Standard:SOT23-3; symbol Simulation_SPICE:NPN -> SparkFun-DiscreteSemi:Q_NPN_BEC
- U8: footprint Package_LGA:LGA-14_3x2.5mm_P0.5mm_LayoutBorder3x4y -> ICM-42688P-HXY 符号:
Connections:
- net +3.3V is gone; now on net 3.3V: R24.2, R31.2, R32.2, U1.9
- net PWM0_P6 is gone; now on net +5V: D15.4 (VDD)
- net +5V: now also C74.1, D10.1 (K), H1.2, MLT-1.1 (+), H10.1, H11.1, H12.1; no longer D15.1 (VDD), H2.2
- net 3.3V: now also C54.1, U7.8 (VCC); no longer C74.1, D10.1 (K), MLT-1.1 (+)
- net DBUS: now also H1.3; no longer H2.3
- net GND: now also D15.2 (VSS), C54.2, D13.1 (A1), D17.1 (A1), D18.1 (A1), D19.1 (A1), H10.2, H10.MP, H11.2, H11.MP, H12.2, H12.MP, H13.MP, H14.MP, H15.MP, H16.MP, R25.1, R26.1, U7.4 (GND); no longer D15.3 (VSS)
- net JTAG_TCK: now also U1.7; no longer U1.3
- net JTAG_TDI: now also R32.1, U1.3; no longer R31.1, U1.1
- net JTAG_TDO: now also U1.4; no longer U1.5
- net JTAG_TMS: now also R31.1, U1.6; no longer R32.1, U1.2
- net JTAG_TRST: now also U1.5; no longer U1.4
- net PWM0_P2: now also D15.3 (DIN); no longer R29.2
- net UART0_RX: now also D29.2 (A2), F21.2; no longer D30.2 (A2), F20.2
- net UART0_TX: now also D30.2 (A2), F20.2; no longer D29.2 (A2), F21.2
- net UART2_RX: now also D17.2 (A2), F18.1; no longer Q2.3 (C), R24.1
- net UART4_RX: now also D14.2 (A2), F14.1; no longer D11.2 (A2), F15.1
- net UART4_TX: now also D16.2 (A2), F13.1; no longer D12.2 (A2), F16.1
- net UART6_RX: now also D12.2 (A2), F16.1; no longer D14.2 (A2), F14.1
- net UART6_TX: now also D11.2 (A2), F15.1; no longer D16.2 (A2), F13.1
- net at R49.1, U10.6 (CANL): now also L5.1; no longer L5.2
- net at R49.2, U10.7 (CANH): now also L5.2; no longer L5.1
- net at D24.1 (K), F9.1: now also L6.3; no longer L6.4
- net at F20.1: now also U1.2; no longer U1.6
- net at F21.1: now also U1.1; no longer U1.7
- net at F15.2: now also H10.3; no longer H1.2
- net at F16.2: now also H10.4; no longer H1.3
- net at R29.1, R30.1: no longer Q3.1 (B)
- net at R50.2, U11.7 (CANH): now also L6.2; no longer L6.1
- net at R50.1, U11.6 (CANL): now also L6.1; no longer L6.2
- net at D24.2 (K), F10.1: now also L6.4; no longer L6.3
- net at F4.1, L7.3: now also D25.2 (K); no longer D25.1 (K)
- net at F3.1, L7.4: now also D25.1 (K); no longer D25.2 (K)
- net at D23.1 (K), F7.1: now also L5.3; no longer L5.4
- net at D23.2 (K), F8.1: now also L5.4; no longer L5.3
- net PWM0_P3 renamed PWM0_P4
- net SPI1_CS renamed SPI3_CS
- net SPI1_MISO renamed SPI3_MISO
- net SPI1_MOSI renamed SPI3_MOSI
- net SPI1_SCLK renamed SPI3_SCLK
- net User_Key renamed SPI2_CS
- net SPI2_CS: now also U7.1 (~{CS})
- new net: F19.2, H12.3
- new net: F22.2, H12.4
- new net: F18.2, H11.4
- new net: F17.2, H11.3
- new net BOOT0: R25.2
- new net BOOT1: R26.2
- new net PWM0_P1: R29.2
- new net SPI2_D2: U7.3 (~{WP}/IO_{2})
- new net SPI2_D3: U7.7 (~{HOLD}/~{RESET}/IO_{3})
- new net SPI2_MISO: U7.2 (DO/IO_{1})
- new net SPI2_MOSI: U7.5 (DI/IO_{0})
- new net SPI2_SCLK: U7.6 (CLK)
- new net UART1_RX: H2.3
- new net UART1_TX: H2.2
- new net UART2_TX: D13.2 (A2), F17.1
- new net UART3_RX: D19.2 (A2), F22.1
- new net UART3_TX: D18.2 (A2), F19.1
- new net UART5_RX: Q2.3 (C), R24.1
Other:
- note added: "RESET&BOOT"
- note added: "UART1"
- note added: "UART2"
- note added: "UART3"
- note removed: "RESET&User_Key"
- moved on the sheet: C64, C65, C66, C67, C68, C69, C70, C71, C72, C75, D11, D12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
