File: hardware/phy.kicad_sch (KiCad schematic)
At the start: 56 parts, among them U2 1789288892504, Y3 25M

Commit message: Update HPM5E31 hardware design and manufacturing files
Parts:
- removed C55, C56: 12pF, Capacitor_SMD:C_0402_1005Metric, symbol SparkFun-Capacitor:C_Small
- removed C57, C58, C59, C60, C61: 100nF, Capacitor_SMD:C_0402_1005Metric, symbol SparkFun-Capacitor:C_Small
- removed C62, C63: 470nF, Capacitor_SMD:C_0402_1005Metric, symbol SparkFun-Capacitor:C_Small
- removed C77: 10nF, Capacitor_SMD:C_0402_1005Metric, symbol SparkFun-Capacitor:C_Small
- removed C86, C87: 10pF, Capacitor_SMD:C_0402_1005Metric, symbol SparkFun-Capacitor:C_Small
- removed D4: LED_E, LED_SMD:LED_0402_1005Metric, symbol Device:LED
- removed D5: LED_G, LED_SMD:LED_0402_1005Metric, symbol Device:LED
- removed L13: 3416自耦环, Inductor_SMD:L_CommonMode_Wurth_WE-CNSW-1206, symbol Device:L_Iron_Coupled
- removed R17: 2.49K, Resistor_SMD:R_0402_1005Metric, symbol Device:R_Small
- removed R25, R26, R27: 10K, Resistor_SMD:R_0402_1005Metric, symbol Device:R_Small
- removed R35: 1K, Resistor_SMD:R_0402_1005Metric, symbol Device:R_Small
- removed Y3: 25M, Crystal:Crystal_SMD_2016-4Pin_2.0x1.6mm, symbol Device:Crystal_GND24
- added C100, C101, C102, C103, C92, C93, C94, C95, C96, C97, C99: 100nF, SparkFun-Capacitor:C_0603_1608Metric, symbol SparkFun-Capacitor:C_Small
- added C98: 470nF, SparkFun-Capacitor:C_0603_1608Metric, symbol SparkFun-Capacitor:C_Small
- added D8: LED_G, LED_SMD:LED_0402_1005Metric, symbol Device:LED
- added R53, R54, R55, R56, R58, R59, R60, R63: 10K, Resistor_SMD:R_0402_1005Metric, symbol Device:R_Small
- added R57: 2.49K, Resistor_SMD:R_0402_1005Metric, symbol Device:R_Small
- added R61: 4.7K, Resistor_SMD:R_0402_1005Metric, symbol Device:R_Small
- added R62: 330R, Resistor_SMD:R_0402_1005Metric, symbol Device:R_Small
- added U3: RTL8201F-VB-CG, kicad_api_lib:RTL8201F-VB-CG, symbol RTL8201F-VB-CG:RTL8201F-VB-CG
- C78, C79, C80, C81, C82, C83, C84, C85, C88, C89, C90, C91: footprint Capacitor_SMD:C_0402_1005Metric -> SparkFun-Capacitor:C_0603_1608Metric
- H3: footprint Connector_JST:JST_PH_B4B-PH-K_1x04_P2.00mm_Vertical -> Connector_JST:JST_GH_BM04B-GHS-TBT_1x04-1MP_P1.25mm_Vertical
- H4: footprint Connector_JST:JST_PH_B2B-PH-K_1x02_P2.00mm_Vertical -> Connector_JST:JST_GH_BM02B-GHS-TBT_1x02-1MP_P1.25mm_Vertical
- L12: footprint Inductor_SMD:L_CommonModeChoke_Coilcraft_0805USB -> Inductor_SMD:L_CommonModeChoke_Coilcraft_1812CAN
- U2: value 1789288892504 -> TJA1101B
Connections:
- net ETH0_MDC is gone; now on net ESC0_MDC: R16.1, U2.1 (MDC)
- net ETH0_MDIO is gone; now on net ESC0_MDIO: R15.1, U2.36 (MDIO)
- net 3.3V: now also U2.10 (INH), U2.11 (VDDA(TX)), U2.14 (VDDA(TX)), U2.15 (VDDD(3V3)), U2.7 (VDDA(3V3)), U2.9 (V_BAT), C100.1, C101.1, C92.1, C93.2, C94.2, C95.2, C96.2, C97.2, C99.1, D8.2 (A), R53.1, R54.1, R55.1, R61.1, R63.1, U3.14 (DVDD33), U3.30 (AVDD33), U3.7 (AVDD33)
- net ENET_PHY_LED0: now also U3.24 (LED0/PHYAD0/PMEB)
- net ENET_PHY_LED1: now also R61.2, R62.2, U3.25 (LED1/PHYAD1)
- net ESC0_MDC: now also U3.22 (MDC)
- net ESC0_MDIO: now also U3.23 (MDIO)
- net ESC0_P1_RXDV: now also U2.18 (RXDV/CONFIG2/CRSDV), R58.2
- net ESC0_P1_RXER: now also U2.17 (RXER/CONFIG3/TXCLK), R59.2
- net ESC0_P1_TXCK: now also U2.28 (TXC)
- net ESC0_REFCK: now also U3.32 (CKXTAL2)
- net GND: now also U2.37 (EP), U2.4 (SEL_1V8), C100.2, C101.2, C102.2, C103.2, C92.2, C93.1, C94.1, C95.1, C96.1, C97.1, C98.1, C99.2, R56.1, R57.1, R58.1, R59.1, R60.1, U3.31 (CKXTAL1), U3.33 (EP); no longer U2.17 (RXER/CONFIG3/TXCLK), U2.18 (RXDV/CONFIG2/CRSDV)
- net TRX_P: now also L12.1; no longer C89.1
- net RX_N: now reaches C89.2
- net RX_N: now also H4.1; no longer L12.1
- net at U2.16 (VDDD(1V8)): now also C98.2
- net ETH0_INT: now reaches U2.2 (~{INT_N})
- net ETH0_INT: now also R53.2
- net ETH0_RESET: now reaches U2.3 (~{RST_N})
- net ETH0_RESET: now also R54.2
- net at U2.34 (TXER): now also R56.2
- net at U2.35 (EN): now also R55.2
- net at C81.2: now also L9.1; no longer L9.4
- net at L12.4: now also C88.1; no longer C88.2
- net at C80.2: now also L9.4; no longer L9.1
- net TRX_N: now reaches L12.2
- net TRX_N: now also U2.13 (TRX_M); no longer H4.1
- net at L12.3: now also C89.1; no longer H4.2
- net RD_N renamed MDI+1
- net MDI+1: now also C78.1, U3.5 (MDI+1); no longer C79.1
- net RD_P renamed MDI-1
- net MDI-1: now also C79.1, U3.6 (MDI-1); no longer C78.1
- net TD_N renamed MDI+0
- net MDI+0: now also C83.1, U3.3 (MDI+0); no longer C82.1
- net TD_P renamed MDI-0
- net MDI-0: now also C82.1, U3.4 (MDI-0); no longer C83.1
- removed net TRX_M: C88.1, U2.13 (TRX_M)
- new net: D8.1 (K), R62.1
- new net: R57.2, U3.1 (RSET)
- new net: C102.1, U3.2 (AVDD10OUT)
- new net: C103.1, U3.29 (DVDD10OUT)
- new net COL: U3.27 (COL)
- new net CRS: U3.26 (CRS/CRS_DV)
- new net ESC0_P0_RXCK: U3.13 (RXC)
- new net ESC0_P0_RXD0: U3.9 (RXD0)
- new net ESC0_P0_RXD1: U3.10 (RXD1)
- new net ESC0_P0_RXD2: U3.11 (RXD2/INTB)
- new net ESC0_P0_RXD3: U3.12 (RXD3/CLK_CTL)
- new net ESC0_P0_RXDV: R60.2, U3.8 (RXDV)
- new net ESC0_P0_RXER: U3.28 (RXER/FXEN)
- new net ESC0_P0_TXCK: U3.15 (TXC)
- new net ESC0_P0_TXD0: U3.16 (TXD0)
- new net ESC0_P0_TXD1: U3.17 (TXD1)
- new net ESC0_P0_TXD2: U3.18 (TXD2)
- new net ESC0_P0_TXD3: U3.19 (TXD3)
- new net ESC0_P0_TXEN: U3.20 (TXEN)
- new net PHYRSTB: R63.2, U3.21 (PHYRSTB)
- new net TX_P: C88.2, H4.2
Other:
- note added: "配置为0"
- note added: "配置为1"
- moved on the sheet: C78, C79, C80, C81, C82, C83, C84, C85, C90, D6, D7, H3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
