File: hardware/usb&crysta.kicad_sch (KiCad schematic)
At the start: 21 parts, among them J1 USB_C_Receptacle_USB2.0_16P, U6 USBLC6-2SC6, U7 HPM5E3YIVK1, Y1 24M

Commit message: Update HPM5E31 hardware design and manufacturing files
Parts:
- removed C34: 100nF, Capacitor_SMD:C_0402_1005Metric, symbol SparkFun-Capacitor:C_Small
- removed U7: HPM5E3YIVK1, Library:BGA-121_11x11_9.0x9.0mm_P0.8mm, symbol HPM5E00_Library:HPM5E3YIVK1
- added R18: 10R, Resistor_SMD:R_0402_1005Metric, symbol Device:R
- added U14: HPM5E31IGN1, HPM_footprints:BGA-196_14x14_12.0x12.0mm_P0.8mm, symbol HPM5E00_Library:HPM5E31IGN1
- C32, C33, C35, C36, C37, C38, C39, C40, C41, C43, C44: footprint Capacitor_SMD:C_0402_1005Metric -> SparkFun-Capacitor:C_0603_1608Metric
Connections:
- net GND: now also J1.SH (SHIELD); no longer J1.S1 (SHIELD)
- net RESET: now also U14.M3 (RSTN)
- net USB_DN: now also U14.L13 (USB0_DN)
- net USB_DP: now also U14.L14 (USB0_DP)
- net VBUS: now also R18.1
- net at C36.2, C37.2: now also U14.J6 (VDD_PHY0CAP)
- net at C38.2, C39.2: now also U14.H6 (VDD_PHY1CAP)
- net at C40.1, R12.2, Y1.1: now also U14.K13 (XTALO)
- net at C41.2, R12.1, Y1.3: now also U14.K14 (XTALI)
- net at C35.2: now also U14.K8 (VDD_OTPCAP)
- net at C32.2, C33.2: now also U14.K7 (VDD_PMCCAP)
- net at R13.1: now also U14.L3 (WKUP)
- net +3.3V renamed 3.3V
- net 3.3V: now also U14.N4 (VPMC), U14.P4 (VPMC)
- new net: R18.2, U14.L12 (USB0_VBUS)
Other:
- moved on the sheet: C32, C33
